File: hackpad.kicad_sch (KiCad schematic)
At the start: 3 parts, among them SW1 SW_Push, U1 XIAO-RP2040-DIP

Commit message: second commit
Parts:
- added D2: SK6812MINI, LED_SMD:LED_SK6812MINI_PLCC4_3.5x3.5mm_P1.75mm, symbol LED:SK6812MINI
- added SW2, SW3, SW4: SW_Push, Button_Switch_Keyboard:SW_Cherry_MX_1.00u_PCB, symbol Switch:SW_Push
- SW1: footprint (none) -> Button_Switch_Keyboard:SW_Cherry_MX_1.00u_PCB
Connections:
- net at U1.10 (GPIO4/MISO): now also SW3.2
- net at U1.11 (GPIO3/MOSI): now also SW4.2
- net GND: now reaches U1.13 (GND)
- net GND: now also D1.2 (VSS), SW1.1, D2.2 (VSS), SW2.1, SW3.1, SW4.1
- net +5V: now reaches U1.14 (VBUS)
- net +5V: now also D1.4 (VDD), D2.4 (VDD)
- net at U1.5 (GPIO6/SDA): now also D1.3 (DIN)
- net at U1.8 (GPIO1/RX): now also SW1.2
- net at U1.9 (GPIO2/SCK): now also SW2.2
- net at D1.1 (DOUT): now also D2.3 (DIN)
Other:
- moved on the sheet: D1, U1

Commit message: fourth commit, why did it not freakin save
Parts:
- added D3, D4: SK6812MINI, LED_SMD:LED_SK6812MINI_PLCC4_3.5x3.5mm_P1.75mm, symbol LED:SK6812MINI
- U1: footprint Module:MOUDLE14P-XIAO-DIP-SMD -> OPL:XIAO-RP2040-DIP
Connections:
- net +5V: now also D3.4 (VDD), D4.4 (VDD)
- net GND: now also D3.2 (VSS), D4.2 (VSS)
- net at D2.1 (DOUT): now also D3.3 (DIN)
- new net: D3.1 (DOUT), D4.3 (DIN)
