File: PCB/_autosave-myproj1.kicad_pcb (KiCad board)
At the start: 2 copper layers, 9 parts, among them SW1 SW_Push, SW2 SW_Push, SW3 SW_Push, SW4 SW_Push, SW5 SW_Coded_SH-7010, U1 XIAO-RP2040-DIP, U3 SHT1x

Commit message: Add files via upload
Parts:
- moved SW1 0.13 mm to (156.9, 96.4)
- moved SW2 0.11 mm to (176.0, 96.4)
- moved SW3 0.06 mm to (156.9, 115.4)
Routing:
- net +5V: vias 1 -> 2
Other:
- board outline added: 56.4 x 67.9 mm
Changed lines of the file:
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@@
 	(footprint "Button_Switch_Keyboard:SW_Cherry_MX_1.00u_PCB"
 		(layer "F.Cu")
-		(at 156.95 96.26)
+		(at 156.89 96.37)
 		(descr "Cherry MX keyswitch, 1.00u, PCB mount, http://cherryamericas.com/wp-content/uploads/2014/12/mx_cat.pdf")
 		(tags "Cherry MX keyswitch 1.00u PCB")
@@
 	(footprint "Button_Switch_Keyboard:SW_Cherry_MX_1.00u_PCB"
 		(layer "F.Cu")
-		(at 176.02 96.26)
+		(at 175.99 96.37)
 		(descr "Cherry MX keyswitch, 1.00u, PCB mount, http://cherryamericas.com/wp-content/uploads/2014/12/mx_cat.pdf")
 		(tags "Cherry MX keyswitch 1.00u PCB")
@@
 	(footprint "Button_Switch_Keyboard:SW_Cherry_MX_1.00u_PCB"
 		(layer "F.Cu")
-		(at 156.95 115.36)
+		(at 156.94 115.42)
 		(descr "Cherry MX keyswitch, 1.00u, PCB mount, http://cherryamericas.com/wp-content/uploads/2014/12/mx_cat.pdf")
 		(tags "Cherry MX keyswitch 1.00u PCB")
@@
 	)
 	(gr_rect
-		(start 137.2 70)
-		(end 190.5 135.7)
+		(start 136.3 70)
+		(end 192.75 137.95)
 		(stroke
-			(width 0.2)
+			(width 0.05)
 			(type default)
 		)
 		(fill no)
-		(layer "F.Cu")
+		(layer "Edge.Cuts")
 	)
 	(gr_text "Xiao here"
@@
 	)
 	(segment
+		(start 143.7 80.6)
+		(end 143.65 80.6)
+		(width 0.2)
+		(layer "F.Cu")
+		(net 1)
+	)
+	(segment
 		(start 141.925 81.725)
 		(end 141.925 81.175)
@@
 	)
 	(segment
+		(start 144 80.3)
+		(end 143.7 80.6)
+		(width 0.2)
+		(layer "F.Cu")
+		(net 1)
+	)
+	(segment
 		(start 141.925 81.175)
 		(end 142.1 81)
@@
 		(start 149.325 82.575)
 		(end 149.325 83.05)
-		(width 0.2)
-		(layer "F.Cu")
-		(net 1)
-	)
-	(segment
-		(start 144 80.3)
-		(end 143.7 80.6)
 		(width 0.2)
 		(layer "F.Cu")
@@
 		(net 1)
 	)
+	(via
+		(at 143.65 80.6)
+		(size 0.6)
+		(drill 0.3)
+		(layers "F.Cu" "B.Cu")
+		(net 1)
+	)
+	(segment
+		(start 143.25 81)
+		(end 143.65 80.6)
+		(width 0.2)
+		(layer "B.Cu")
+		(net 1)
+	)
 	(segment
 		(start 142.349 81)
-		(end 143.3 81)
+		(end 143.25 81)
 		(width 0.2)
 		(layer "B.Cu")
-		(net 1)
-	)
-	(segment
-		(start 143.3 81)
-		(end 143.7 80.6)
-		(width 0.2)
-		(layer "B.Cu")
