File: PCB/myproj1b.kicad_sch (KiCad schematic)
At the start: 9 parts, among them SW1 SW_Push, SW2 SW_Push, SW3 SW_Push, SW4 SW_Push, SW5 SW_Coded_SH-7010, U1 XIAO-RP2040-DIP, U3 SHT1x

Commit message: Add files via upload
Parts:
- SW5: footprint Button_Switch_SMD:Nidec_Copal_SH-7010A -> (none)
Changed lines of the file:
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@@
 			)
 		)
-		(property "Footprint" "Button_Switch_SMD:Nidec_Copal_SH-7010A"
+		(property "Footprint" ""
 			(at 110.49 64.77 0)
 			(effects
